File: Envelope/EnvGen.sch (KiCad schematic (older format))
At the start: 36 parts, among them J1 Input, J2 Output, J3 Power, Q1 BC817, Q2 BC817, Q3 BC817, U1 NE555, U2 LM324A

Commit message: New edit schems, add net lists, pcb files and library
Parts:
- C1, C2, C4, C5: symbol device:C -> Device:C
- C3: symbol device:CP -> Device:CP
- D1, D2, D3, D4, D5, D6: symbol device:D -> Device:D
- J1: symbol conn:Conn_01x02_Male -> Connector:Conn_01x02_Male
- J2, J3: symbol conn:Conn_01x03_Male -> Connector:Conn_01x03_Male
- Q1, Q2, Q3: symbol transistors:BC817 -> Transistor_BJT:BC817
- R1, R10, R11, R12, R13, R2, R3, R4, R5, R6, R7, R8, R9: symbol device:R -> Device:R
- RV1, RV2, RV3, RV4: footprint Potentiometer_THT:Potentiometer_Bourns_PTV09A-1_Single_Vertical -> R0409N:PTV09A4020FB103; symbol device:POT -> Device:R_POT
- U1: symbol linear:NE555 -> Timer:NE555
- U2: symbol linear:LM324 -> Amplifier_Operational:LM324
Connections:
- net +5V: no longer U2.11 (V-)
- net -5V: no longer U2.4 (V+)
Changed lines of the file:
@@
 EESchema Schematic File Version 4
-LIBS:EnvGen-cache
 EELAYER 26 0
 EELAYER END
@@
 $EndDescr
 $Comp
-L conn:Conn_01x02_Male J1
+L Connector:Conn_01x02_Male J1
 U 1 1 5C8ABD55
 P 1100 2750
@@
 $EndComp
 $Comp
-L device:D D2
+L Device:D D2
 U 1 1 5C8ABDE0
 P 1600 2550
@@
 $EndComp
 $Comp
-L device:D D5
+L Device:D D5
 U 1 1 5C8ABE20
 P 1600 2950
@@
 $EndComp
 $Comp
-L device:R R9
+L Device:R R9
 U 1 1 5C8ABE65
 P 1950 2750
@@
 $EndComp
 $Comp
-L transistors:BC817 Q1
+L Transistor_BJT:BC817 Q1
 U 1 1 5C8ABF37
 P 2350 2750
@@
 $EndComp
 $Comp
-L device:R R2
+L Device:R R2
 U 1 1 5C8ABF70
 P 2450 2300
@@
 $EndComp
 $Comp
-L device:R R6
+L Device:R R6
 U 1 1 5C8ABFAD
 P 2750 2450
@@
 $EndComp
 $Comp
-L transistors:BC817 Q2
+L Transistor_BJT:BC817 Q2
 U 1 1 5C8AC01E
 P 3150 2750
@@
 $EndComp
 $Comp
-L device:R R3
+L Device:R R3
 U 1 1 5C8AC061
 P 3250 2300
@@
 $EndComp
 $Comp
-L device:C C1
+L Device:C C1
 U 1 1 5C8AC0A6
 P 3700 2450
@@
 $EndComp
 $Comp
-L device:D D3
+L Device:D D3
 U 1 1 5C8AC0F8
 P 4000 2700
@@
 $EndComp
 $Comp
-L device:R R7
+L Device:R R7
 U 1 1 5C8AC195
 P 4300 2450
@@
 $EndComp
 $Comp
-L transistors:BC817 Q3
+L Transistor_BJT:BC817 Q3
 U 1 1 5C8AC705
 P 4750 2750
@@
 $EndComp
 $Comp
-L device:R R4
+L Device:R R4
 U 1 1 5C8AC758
 P 4850 2400
@@
 $EndComp
 $Comp
-L linear:NE555 U1
+L Timer:NE555 U1
 U 1 1 5C8AC7D6
 P 6300 2750
@@
 Connection ~ 4850 1900
 $Comp
-L device:C C2
+L Device:C C2
 U 1 1 5C8B0FDC
 P 5350 2900
@@
 	3450 2450 3250 2450
 $Comp
-L device:POT RV1
+L Device:R_POT RV1
 U 1 1 5C8B3028
 P 7850 2300
 F 0 "RV1" V 8050 2550 50  0000 C CNN
 F 1 "100K" V 7950 2550 50  0000 C CNN
-F 2 "Potentiometer_THT:Potentiometer_Bourns_PTV09A-1_Single_Vertical" H 7850 2300 50  0001 C CNN
+F 2 "R0409N:PTV09A4020FB103" H 7850 2300 50  0001 C CNN
 F 3 "~" H 7850 2300 50  0001 C CNN
 F 4 "R-0904N-B100K" V 7750 2300 50  0000 C CNN "Тип"
@@
 $EndComp
 $Comp
-L device:POT RV2
+L Device:R_POT RV2
 U 1 1 5C8B3122
 P 7850 2800
 F 0 "RV2" V 8000 3100 50  0000 C CNN
 F 1 "100K" V 7900 3100 50  0000 C CNN
-F 2 "Potentiometer_THT:Potentiometer_Bourns_PTV09A-1_Single_Vertical" H 7850 2800 50  0001 C CNN
+F 2 "R0409N:PTV09A4020FB103" H 7850 2800 50  0001 C CNN
 F 3 "~" H 7850 2800 50  0001 C CNN
 F 4 "R-0904N-B100K" V 7750 2850 50  0000 C CNN "Тип"
@@
 $EndComp
 $Comp
-L device:POT RV4
+L Device:R_POT RV4
 U 1 1 5C8B31B5
 P 7800 3250
 F 0 "RV4" V 7700 3250 50  0000 C CNN
 F 1 "100K" V 7750 3000 50  0000 C CNN
-F 2 "Potentiometer_THT:Potentiometer_Bourns_PTV09A-1_Single_Vertical" H 7800 3250 50  0001 C CNN
+F 2 "R0409N:PTV09A4020FB103" H 7800 3250 50  0001 C CNN
 F 3 "~" H 7800 3250 50  0001 C CNN
 F 4 "R-0904N-B100K" V 7600 3200 50  0000 C CNN "Тип"
@@
 $EndComp
 $Comp
-L device:POT RV3
+L Device:R_POT RV3
 U 1 1 5C8B3251
 P 7350 3050
 F 0 "RV3" H 7280 3141 50  0000 R CNN
 F 1 "10K" H 7280 3050 50  0000 R CNN
-F 2 "Potentiometer_THT:Potentiometer_Bourns_PTV09A-1_Single_Vertical" H 7350 3050 50  0001 C CNN
+F 2 "R0409N:PTV09A4020FB103" H 7350 3050 50  0001 C CNN
 F 3 "~" H 7350 3050 50  0001 C CNN
 F 4 "R-0904N-B10K" H 7600 2800 50  0000 R CNN "Тип"
@@
 $EndComp
 $Comp
-L device:D D1
+L Device:D D1
 U 1 1 5C8B32B2
 P 8200 2300
@@
 $EndComp
 $Comp
-L device:D D4
+L Device:D D4
 U 1 1 5C8B3304
 P 8200 2800
@@
 $EndComp
 $Comp
-L device:D D6
+L Device:D D6
 U 1 1 5C8B3360
 P 8200 3100
@@
 $EndComp
 $Comp
-L device:R R5
+L Device:R R5
 U 1 1 5C8B33BD
 P 8550 2300
@@
 $EndComp
 $Comp
-L device:R R10
+L Device:R R10
 U 1 1 5C8B3464
 P 8550 2800
@@
 $EndComp
 $Comp
-L device:R R12
+L Device:R R12
 U 1 1 5C8B34DE
 P 8550 3100
@@
 $EndComp
 $Comp
-L device:R R1
+L Device:R R1
 U 1 1 5C8B355B
 P 6550 1900
@@
 Connection ~ 8800 3100
 $Comp
-L device:CP C3
+L Device:CP C3
 U 1 1 5C8C67E0
 P 6600 3300
@@
 $EndComp
 $Comp
-L linear:LM324 U2
+L Amplifier_Operational:LM324 U2
 U 1 1 5C8E0A0F
 P 9200 2950
@@
 	9500 2450 9500 2950
 $Comp
-L device:R R13
+L Device:R R13
 U 1 1 5C8E7395
 P 9800 3250
@@
 $EndComp
 $Comp
-L device:R R11
+L Device:R R11
 U 1 1 5C8E7401
 P 9800 2950
@@
 $EndComp
 $Comp
-L device:R R8
+L Device:R R8
 U 1 1 5C8EBBC9
 P 9800 2650
@@
 	9650 2950 9650 3250
 $Comp
-L conn:Conn_01x03_Male J2
+L Connector:Conn_01x03_Male J2
 U 1 1 5C8F2C0C
 P 10400 2950
@@
 	7350 3250 7350 3200
 $Comp
-L conn:Conn_01x03_Male J3
+L Connector:Conn_01x03_Male J3
 U 1 1 5CA906B6
 P 2050 4350
@@
 $EndComp
 $Comp
-L device:C C4
+L Device:C C4
 U 1 1 5CA907F6
 P 2900 3800
@@
 $EndComp
 $Comp
-L device:C C5
+L Device:C C5
 U 1 1 5CA9086E
 P 2900 5000
@@
 Wire Wire Line
 	2350 4050 2900 4050
-Connection ~ 2900 4050
-Wire Wire Line
-	2900 4050 2900 4100
-Wire Wire Line
-	2900 4700 2900 4800
 Wire Wire Line
 	2250 4450 2350 4450
@@
 Wire Wire Line
 	2350 4800 2900 4800
-Connection ~ 2900 4800
 Wire Wire Line
 	2900 4800 2900 4850
@@
 Wire Wire Line
 	6300 3150 6300 3300
-Wire Wire Line
-	9100 2650 9100 2150
-Wire Wire Line
-	9100 2150 10850 2150
-Wire Wire Line
-	10850 2150 10850 4100
-Wire Wire Line
-	10850 4100 2900 4100
-Wire Wire Line
-	2900 4700 9100 4700
-Wire Wire Line
-	9100 4700 9100 3250
+Connection ~ 9500 2950
 $EndSCHEMATC

Commit message: Изменены библиотеки. Добавлинны библиотеки примененные в проекте локально. Добавленны заготовки для печатных плат. Добавленны 3D модели компоненток.
Parts:
- C1, C2, C4, C5: footprint Capacitor_SMD:C_0603_1608Metric -> footprint:c0603; symbol Device:C -> uRack:C
- C3: footprint Capacitor_THT:CP_Radial_D4.0mm_P1.50mm -> footprint:cp_5x2_5; symbol Device:CP -> uRack:CP
- D1, D2, D3, D4, D5, D6: footprint Diode_SMD:D_0201_0603Metric -> footprint:d0603; symbol Device:D -> uRack:D
- J1: footprint Connector_PinHeader_2.54mm:PinHeader_1x02_P2.54mm_Vertical -> footprint:pls1x02; symbol Connector:Conn_01x02_Male -> uRack:Conn_01x02_Male
- J2, J3: footprint Connector_PinHeader_2.54mm:PinHeader_1x03_P2.54mm_Vertical -> footprint:pls1x03; symbol Connector:Conn_01x03_Male -> uRack:Conn_01x03_Male
- Q1, Q2, Q3: footprint Package_TO_SOT_SMD:SOT-23 -> footprint:SOT-23; symbol Transistor_BJT:BC817 -> uRack:BC817
- R1, R10, R11, R12, R13, R2, R3, R4, R5, R6, R7, R8, R9: footprint Resistor_SMD:R_0603_1608Metric -> footprint:r0603; symbol Device:R -> uRack:R
- RV1, RV2, RV3, RV4: footprint R0409N:PTV09A4020FB103 -> footprint:R0904N; symbol Device:R_POT -> uRack:R_POT
- U1: footprint Package_SO:SO-8_5.3x6.2mm_P1.27mm -> footprint:soic-8; symbol Timer:NE555 -> uRack:LM555
- U2: footprint Package_SO:SOIC-14_3.9x8.7mm_P1.27mm -> footprint:soic-14; symbol Amplifier_Operational:LM324 -> uRack:LM324
