File: Envelope/EnvGen.sch (KiCad schematic (older format))
At the start: 36 parts, among them J1 Input, J2 Output, J3 Power, Q1 BC817, Q2 BC817, Q3 BC817, U1 NE555, U2 LM324A

Commit message: Изменение в схемах. Разведенны ПП
Parts:
- removed J3: Power, footprint:pls1x03, symbol uRack:Conn_01x03_Male
- added J10, J11, J3, J4, J5, J6, J7, J8, J9: Conn_01x05_Male, footprint:pls1x05, symbol uRack:Conn_01x05_Male
- added unit 5 of U2
- U2: value LM324A -> LM324
- renumbered C5 to C4, C4 to C5, R5 to R4, R4 to R5
Connections:
- wire segments 119 -> 215
