File: Envelope/EnvGen.kicad_pcb (KiCad board)
At the start: 2 copper layers, 36 parts, among them J1 Input, J2 Output, J3 Power, Q1 BC817, Q2 BC817, Q3 BC817, U1 NE555, U2 LM324A

Commit message: Изменение в схемах. Разведенны ПП
Parts:
- added J10: Conn_01x05_Male, footprint:pls1x05, B.Cu at (47.0, 78.0)
- added J11: Conn_01x05_Male, footprint:pls1x05, B.Cu at (72.4, 78.0)
- added J4: Conn_01x05_Male, footprint:pls1x05, B.Cu at (25.4, 24.0)
- added J5: Conn_01x05_Male, footprint:pls1x05, B.Cu at (25.4, 85.0)
- added J6: Conn_01x05_Male, footprint:pls1x05, B.Cu at (73.7, 24.0)
- added J7: Conn_01x05_Male, footprint:pls1x05, B.Cu at (77.7, 85.0)
- added J8: Conn_01x05_Male, footprint:pls1x05, B.Cu at (48.3, 85.0)
- added J9: Conn_01x05_Male, footprint:pls1x05, B.Cu at (24.1, 78.0)
- C1, C2, C4, C5, D1, D2, D3, D4, D5, D6, Q1, Q2, Q3, R1, R10, R11, R12, R13, R2, R3, R6, R7, R8, R9, U1: moved to B.Cu
- J3: value Power -> Conn_01x05_Male; footprint footprint:pls1x03 -> footprint:pls1x05; moved to B.Cu
- R4: value 10K -> 100R; moved to B.Cu
- R5: value 100R -> 10K; moved to B.Cu
- U2: value LM324A -> LM324; moved to B.Cu
- moved D1 132.5 mm to (37.1, 50.1)
- moved Q1 131.7 mm to (34.3, 60.6), turned to 270 degrees
- moved R10 128.4 mm to (44.0, 57.0)
- moved RV1 124.9 mm to (33.8, 40.9)
- moved J1 121.1 mm to (26.6, 55.5)
- moved D2 117.9 mm to (30.6, 55.5), turned to 180 degrees
- moved Q2 117.3 mm to (39.0, 60.5)
- moved R9 115.2 mm to (33.4, 56.2), turned to 90 degrees
- moved R4 110.4 mm to (40.5, 50.1), turned to 180 degrees
- moved C2 109.1 mm to (57.0, 59.6), turned to 90 degrees
- moved D5 108.4 mm to (30.6, 58.1), turned to 180 degrees
- moved R12 107.4 mm to (42.0, 52.9)
- moved J3 106.7 mm to (48.3, 24.0), turned to 270 degrees
- moved D3 106.4 mm to (38.8, 57.4), turned to 180 degrees
- moved R6 103.9 mm to (69.1, 69.7)
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Connections:
- C4 pad 1: GNDREF -> -5V
- C4 pad 2: +5V -> GNDREF
- C5 pad 1: -5V -> GNDREF
- C5 pad 2: GNDREF -> +5V
- J3 pad 1: +5V -> -5V
- J3 pad 2: GNDREF -> -5V
- R4 pad 1: +5V -> Net-(C3-Pad1)
- R4 pad 2: Net-(Q3-Pad3) -> Net-(D1-Pad2)
- R5 pad 1: Net-(C3-Pad1) -> +5V
- R5 pad 2: Net-(D1-Pad2) -> Net-(Q3-Pad3)
- U2 pad 11: (no net) -> +5V
- U2 pad 4: (no net) -> -5V
Routing:
- net GNDREF: track 0.00 -> 206.5 mm, vias 0 -> 5
- net -5V: track 0.00 -> 147.8 mm, vias 0 -> 1
- net +5V: track 0.00 -> 126.6 mm, vias 0 -> 4
- net Net-(C1-Pad2): track 0.00 -> 82.5 mm, vias 0 -> 4
- net Net-(C3-Pad1): track 0.00 -> 60.0 mm, vias 0 -> 5
- net Net-(Q1-Pad3): track 0.00 -> 57.9 mm, vias 0 -> 2
- net Net-(D6-Pad1): track 0.00 -> 57.1 mm
- net Net-(Q3-Pad3): track 0.00 -> 53.4 mm, vias 0 -> 2
- net Net-(C1-Pad1): track 0.00 -> 45.6 mm, vias 0 -> 2
- net Net-(R11-Pad1): track 0.00 -> 40.9 mm, vias 0 -> 2
- net Net-(Q2-Pad1): track 0.00 -> 39.5 mm, vias 0 -> 2
- net Net-(RV3-Pad3): track 0.00 -> 32.8 mm, vias 0 -> 1
- net Net-(RV2-Pad1): track 0.00 -> 29.1 mm
- net Net-(RV3-Pad2): track 0.00 -> 19.6 mm
- net Net-(D4-Pad1): track 0.00 -> 13.7 mm
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Other:
- board outline added: 80 x 70 mm
- net class power added: clearance 0.2, trace_width 0.5, via_dia 0.8, via_drill 0.4
