File: VCA/VCA.sch (KiCad schematic (older format))
At the start: 36 parts, among them J1 Output, J2 Input, J3 Power, J4 Env, Q1 BC817, Q2 BC817, Q3 BC817, Q4 BC817, Q5 BC807, U1 LM324A

Commit message: New edit schems, add net lists, pcb files and library
Parts:
- removed U1: LM324A, Package_SO:SOIC-14_3.9x8.7mm_P1.27mm, symbol VCA-rescue:LM324A-Amplifier_Operational
- added U1: LM324, Package_SO:SOIC-14_3.9x8.7mm_P1.27mm, symbol Amplifier_Operational:LM324
- C1, C2: footprint Capacitors_SMD:C_0603 -> Capacitor_SMD:C_0603_1608Metric; symbol VCA-rescue:C-Device -> Device:C
- J1, J2, J3, J4: symbol VCA-rescue:Conn_01x03_Male-Connector -> Connector:Conn_01x03_Male
- Q1, Q2, Q3, Q4: footprint TO_SOT_Packages_SMD:SOT-23 -> Package_TO_SOT_SMD:SOT-23; symbol VCA-rescue:BC817-Transistor_BJT -> Transistor_BJT:BC817
- Q5: footprint TO_SOT_Packages_SMD:SOT-23 -> Package_TO_SOT_SMD:SOT-23; symbol VCA-rescue:BC807-Transistor_BJT -> Transistor_BJT:BC807
- R1, R10, R11, R12, R13, R14, R15, R16, R17, R18, R19, R2, R20, R21, R22, R3, R4, R5, R6, R7: footprint Resistors_SMD:R_0603 -> Resistor_SMD:R_0603_1608Metric; symbol VCA-rescue:R-Device -> Device:R
- R8: renamed from R9; footprint Resistors_SMD:R_0603 -> Resistor_SMD:R_0603_1608Metric; symbol VCA-rescue:R-Device -> Device:R
- R9: renamed from R8; footprint Resistors_SMD:R_0603 -> Resistor_SMD:R_0603_1608Metric; symbol VCA-rescue:R-Device -> Device:R
- RV1, RV2: footprint Potentiometers:Potentiometer_Bourns_PTV09A-1_Horizontal -> R0409N:PTV09A4020FB103; symbol VCA-rescue:R_POT-Device -> Device:R_POT
Connections:
- net +5V: now also U1.4 (V+)
- net -5V: now also U1.11 (V-)
- net at R10.1, R5.1, R7.1: now also U1.2 (-)
- net at RV1.2: now also U1.3 (+)
- net at R9.2, RV1.3: now also U1.1
- net at Q1.3 (C), R1.2, R2.2: now also U1.6 (-)
- net at Q2.3 (C), R11.1, R3.2: now also U1.5 (+)
- net at R1.1, R4.2, R6.2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: now also U1.7
- net at R16.1, R18.1, R19.1: now also U1.9 (-)
- net at R17.2, RV2.3: now also U1.8
- net at RV2.2: now also U1.10 (+)

Commit message: Изменены библиотеки. Добавлинны библиотеки примененные в проекте локально. Добавленны заготовки для печатных плат. Добавленны 3D модели компоненток.
Parts:
- C1, C2: footprint Capacitor_SMD:C_0603_1608Metric -> footprint:c0603; symbol Device:C -> uRack:C
- J1, J2, J3, J4: footprint Connector_PinHeader_2.54mm:PinHeader_1x03_P2.54mm_Vertical -> footprint:pls1x03; symbol Connector:Conn_01x03_Male -> uRack:Conn_01x03_Male
- Q1, Q2, Q3, Q4: footprint Package_TO_SOT_SMD:SOT-23 -> footprint:SOT-23; symbol Transistor_BJT:BC817 -> uRack:BC817
- Q5: footprint Package_TO_SOT_SMD:SOT-23 -> footprint:SOT-23; symbol Transistor_BJT:BC807 -> uRack:BC807
- R1, R10, R11, R12, R13, R14, R15, R16, R17, R18, R19, R2, R20, R21, R22, R3, R4, R5, R6, R7, R8, R9: footprint Resistor_SMD:R_0603_1608Metric -> footprint:r0603; symbol Device:R -> uRack:R
- RV1, RV2: footprint R0409N:PTV09A4020FB103 -> footprint:PTV09A4020FB103; symbol Device:R_POT -> uRack:R_POT
- U1: footprint Package_SO:SOIC-14_3.9x8.7mm_P1.27mm -> footprint:soic-14; symbol Amplifier_Operational:LM324 -> uRack:LM324
- U1: footprint Package_SO:SOIC-14_3.9x8.7mm_P1.27mm -> footprint:soic-14

Commit message: fix relative path, fix lib path in VCO
Parts:
- U1: symbol Amplifier_Operational:LM324 -> uRack:LM324
Changed lines of the file:
@@
 Connection ~ 6950 1700
 $Comp
-L Amplifier_Operational:LM324 U1
+L uRack:LM324 U1
 U 1 1 5C794BC3
 P 4200 1950
