File: VCA/VCA.sch (KiCad schematic (older format))
At the start: 36 parts, among them J1 Output, J2 Input, J3 Power, J4 Env, Q1 BC817, Q2 BC817, Q3 BC817, Q4 BC817, Q5 BC807, U1 LM324

Commit message: Изменение в схемах. Разведенны ПП
Parts:
- removed J3: Power, footprint:pls1x03, symbol uRack:Conn_01x03_Male
- added J10, J11, J12, J4, J5, J6, J7, J8, J9: Conn_01x05_Male, footprint:pls1x05, symbol uRack:Conn_01x05_Male
- RV1, RV2: footprint footprint:PTV09A4020FB103 -> footprint:R0904N
- renumbered J4 to J3
Connections:
- wire segments 134 -> 223
Other:
- moved on the sheet: C1, C2, U1E
