File: VCF/VCF.sch (KiCad schematic (older format))
At the start: 33 parts, among them J1 Env, J2 Power, J3 Output, J4 Input, U1 LM324A

Commit message: Изменение в схемах. Разведенны ПП
Parts:
- removed J2: Power, footprint:pls1x03, symbol uRack:Conn_01x03_Male
- added J1, J10, J12, J2, J4, J5, J6, J7, J8: Conn_01x05_Male, footprint:pls1x05, symbol uRack:Conn_01x05_Male
- RV1, RV2, RV3: footprint footprint:PTV09A4020FB103 -> footprint:R0904N
- renumbered J4 to J11, J1 to J3, J3 to J9
Connections:
- wire segments 123 -> 208
Other:
- moved on the sheet: C1, C2, U1E
